File: schema elettrificato/smistarumori.kicad_sch (KiCad schematic)
At the start: 33 parts, among them J1 SSD1306, J2 LCD RETROILLUMINAZIONE, J3 Relay module, Q1 2N3906, SW1 SW_Push, SW2 SW_Push, SW3 SW_Push, SW4 SW_Push, SW5 SW_Push, SW6 SW_Push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

Commit message: relese 1
Changed lines of the file:
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@@
 		)
 	)
-	(label "In 2 ON GP7=HIGH"
-		(at 54.61 96.52 0)
+	(label "In B ON GP7=HIGH"
+		(at 64.77 96.52 0)
 		(effects
 			(font
@@
 		)
 	)
-	(label "In 1 ON GP6=LOW"
+	(label "In A ON GP6=LOW"
 		(at 81.28 55.88 0)
 		(effects
@@
 		)
 	)
-	(label "In 3 ON GP7=LOW"
+	(label "In C ON GP7=LOW"
 		(at 78.74 105.41 0)
 		(effects
